File: Modxo-Mega/Modxo-Mega.kicad_pcb (KiCad board)
At the start: 2 copper layers, 42 x 50 mm, 50 parts, among them J1 LPC, J2 USB-C, J3 LCD, J4 UART, J5 D0, J6 OXHD, J7 RGB, J8 DBG, J9 EXP I2C, SW1 Boot, U1 RP2040, U2 W25Q128JVS, U3 AP2112K-3.3, X1 12MHz

Commit message: Move most symbols to library
Routing:
- net GND: vias 82 -> 81
Changed lines of the file:
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@@
-	)
-	(via
-		(at 141.79 79.5)
-		(size 0.7)
-		(drill 0.3)
-		(layers "F.Cu" "B.Cu")
-		(free yes)
-		(net "GND")
 	)
 	(via
