File: Modxo-Mega/mcu.kicad_sch (KiCad schematic)
At the start: 31 parts, among them J2 USB-C, SW1 Boot, U1 RP2040, X1 12MHz

Commit message: Cleanup schematic
Parts:
- added C16: 100n, Capacitor_SMD:C_0402_1005Metric, symbol Modxo-Raw:C_100n_0402_Decouple
- added C3, C4: 1u, Resistor_SMD:R_0603_1608Metric, symbol Modxo-Raw:C_1u_0402_Decouple
- added D1: 1N5819WS, Diode_SMD:D_SOD-323, symbol Diode:1N5819WS
- added J1: LPC, Connector_PinSocket_2.54mm:PinSocket_2x08_P2.54mm_Vertical_SMD, symbol Connector_Generic:Conn_02x08_Odd_Even
- added R10: DNP, Resistor_SMD:R_0402_1005Metric, symbol Device:R_Small
- added R3: 1k, Resistor_SMD:R_0402_1005Metric, symbol Modxo-Raw:R_1k_0402
- added U2: W25Q128JVS, Package_SO:SOIC-8_5.3x5.3mm_P1.27mm, symbol Memory_Flash:W25Q128JVS
- added U3: AP2112K-3.3, Package_TO_SOT_SMD:SOT-23-5, symbol Regulator_Linear:AP2112K-3.3
Connections:
- net +3V3: now also C16.1, C4.1, R10.1, U2.8 (VCC), U3.5 (VOUT)
- net +VSYS: now also C3.1, D1.1 (K), U3.1 (VIN), U3.3 (EN)
- net GND: now also C16.2, C3.2, C4.2, J1.12 (Pin_12), J1.2 (Pin_2), U2.4 (GND), U3.2 (GND)
- net LAD0: now also J1.11 (Pin_11)
- net LAD1: now also J1.10 (Pin_10)
- net LAD2: now also J1.8 (Pin_8)
- net LAD3: now also J1.7 (Pin_7)
- net LPC_3V3: now also J1.9 (Pin_9)
- net LPC_LCLK: now also J1.1 (Pin_1)
- net LPC_LFRAME: now also J1.3 (Pin_3)
- net LPC_RST: now also J1.5 (Pin_5)
- net QSPI_SCLK: now also U2.6 (CLK)
- net QSPI_SD0: now also U2.5 (DI/IO_{0})
- net QSPI_SD1: now also U2.2 (DO/IO_{1})
- net QSPI_SD2: now also U2.3 (~{WP}/IO_{2})
- net QSPI_SD3: now also U2.7 (~{HOLD}/~{RESET}/IO_{3})
- net QSPI_SS: now also R10.2, R3.2, U2.1 (~{CS})
- net USB_BOOT: now also R3.1
- new net +LPC_5V: D1.2 (A), J1.6 (Pin_6)
- new net XSMBUS_SCL: J1.13 (Pin_13)
- new net XSMBUS_SDA: J1.14 (Pin_14)
- no-connect marks 13 -> 16
Other:
- note added: "Flash"
- note added: "LPC Header"
- note added: "Voltage Regulator"
- moved on the sheet: C15, LED2, SW1

Commit message: Add SD Card, other minor changes
Parts:
- R10: now not fitted; now left out of the parts list
- R5, R6: Distributor LInk 2 https://www.mouser.com/ProductDetail/Royalohm/0603WAF5101T5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 -> (none); Distributor Link 2 (none) -> https://www.mouser.com/ProductDetail/Royalohm/0603WAF5101T5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
Connections:
- net LAD0R: now also U1.6 (GPIO4); no longer U1.13 (GPIO10)
- net LAD1R: now also U1.7 (GPIO5); no longer U1.14 (GPIO11)
- net LAD2R: now also U1.8 (GPIO6); no longer U1.15 (GPIO12)
- net LAD3R: now also U1.9 (GPIO7); no longer U1.16 (GPIO13)
- net LPC_3V3: now also U1.5 (GPIO3); no longer U1.7 (GPIO5)
- net LPC_LCLK: now also U1.2 (GPIO0); no longer U1.4 (GPIO2)
- net LPC_LFRAME: now also U1.3 (GPIO1); no longer U1.5 (GPIO3)
- net LPC_RST: now also U1.4 (GPIO2); no longer U1.6 (GPIO4)
- net SD_CLK: now reaches U1.11 (GPIO8)
- net SD_CSN: now reaches U1.12 (GPIO9)
- new net SD_MISO: U1.14 (GPIO11)
- new net SD_MOSI: U1.13 (GPIO10)
- no-connect marks 16 -> 12
Other:
- moved on the sheet: RN1

Commit message: Begin saving symbols to library
Parts:
- C17, C18: symbol Device:C_Small -> Modxo-Designs:C_15p_0603_Decouple
- R7: symbol Device:R_Small -> Modxo-Designs:R_470_0603_LED; Distributor Link 1 (none) -> https://www.digikey.com/en/products/detail/yageo/RC0603FR-0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; Distributor Link 2 https://www.mouser.com/ProductDetail/Royalohm/0603WAF4700T5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 -> https://www.mouser.com/en/ProductDetail/YAGEO/RC0603FR-0747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; LCSC C23179 -> C114669; Manufacturer UNI-ROYAL -> Yageo; Manufacturer Part Number 0603WAF4700T5E -> RC0603FR-07470RL
- X1: symbol Device:Crystal_GND24_Small -> Modxo-Designs:ABM8-272-T3
Changed lines of the file:
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@@
 	)
 	(symbol
-		(lib_id "Device:R_Small")
+		(lib_id "Modxo-Designs:R_470_0603_LED")
 		(at 110.49 97.79 90)
 		(unit 1)
@@
 			)
 		)
-		(property "Datasheet" "https://www.lcsc.com/datasheet/C23179.pdf"
+		(property "Datasheet" "https://www.lcsc.com/datasheet/C114669.pdf"
 			(at 110.49 97.79 0)
 			(hide yes)
@@
 			)
 		)
-		(property "Description" "Resistor, small symbol"
+		(property "Description" "470Ω ±1% 100mW 0603 Thick Film Resistor"
 			(at 110.49 97.79 0)
 			(hide yes)
@@
 			)
 		)
-		(property "Manufacturer" "UNI-ROYAL"
+		(property "Manufacturer" "Yageo"
 			(at 110.49 97.79 0)
 			(hide yes)
@@
 			)
 		)
-		(property "Manufacturer Part Number" "0603WAF4700T5E"
+		(property "Manufacturer Part Number" "RC0603FR-07470RL"
 			(at 110.49 97.79 0)
 			(hide yes)
@@
 			)
 		)
-		(property "Distributor Link 1" ""
+		(property "Distributor Link 1" "https://www.digikey.com/en/products/detail/yageo/RC0603FR-07470RL/727256"
 			(at 110.49 97.79 0)
 			(hide yes)
@@
 			)
 		)
-		(property "Distributor Link 2" "https://www.mouser.com/ProductDetail/Royalohm/0603WAF4700T5E?qs=e8oIoAS2J1QEPJMwDZlptQ%3D%3D"
+		(property "Distributor Link 2" "https://www.mouser.com/en/ProductDetail/YAGEO/RC0603FR-07470RL?qs=gt6vzsuosg2Xv5elfMBXPA%3D%3D"
 			(at 110.49 97.79 0)
 			(hide yes)
@@
 			)
 		)
-		(property "LCSC" "C23179"
+		(property "LCSC" "C114669"
 			(at 110.49 97.79 0)
 			(hide yes)
@@
 	)
 	(symbol
-		(lib_id "Device:C_Small")
+		(lib_id "Modxo-Designs:C_15p_0603_Decouple")
 		(at 30.48 120.65 180)
 		(unit 1)
@@
 			)
 		)
-		(property "Description" "Unpolarized capacitor, small symbol"
+		(property "Description" "15pF ±5% 50V Ceramic Capacitor C0G 0603"
 			(at 30.48 120.65 0)
 			(hide yes)
@@
 	)
 	(symbol
-		(lib_id "Device:Crystal_GND24_Small")
+		(lib_id "Modxo-Designs:ABM8-272-T3")
 		(at 24.13 114.3 0)
 		(unit 1)
@@
 			)
 		)
-		(property "Description" "Four pin crystal, GND on pins 2 and 4, small symbol"
+		(property "Description" "12MHz Crystal"
 			(at 24.13 114.3 0)
 			(hide yes)
@@
 	)
 	(symbol
-		(lib_id "Device:C_Small")
+		(lib_id "Modxo-Designs:C_15p_0603_Decouple")
 		(at 17.78 120.65 0)
 		(unit 1)
@@
 			)
 		)
-		(property "Description" "Unpolarized capacitor, small symbol"
+		(property "Description" "15pF ±5% 50V Ceramic Capacitor C0G 0603"
 			(at 17.78 120.65 0)
 			(hide yes)

Commit message: Continue work
Parts:
- R5, R6: symbol Device:R_Small -> Modxo-Designs:R_5k1_0603_USB
- R8, R9: symbol Device:R_Small -> Modxo-Designs:R_27_0402_USB
- RN1: symbol Device:R_Pack04 -> Modxo-Designs:R_Array_100_0603_LPC
Changed lines of the file:
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@@
 	)
 	(symbol
-		(lib_id "Device:R_Pack04")
+		(lib_id "Modxo-Designs:R_Array_100_0603_LPC")
 		(at 113.03 52.07 270)
 		(mirror x)
@@
 			)
 		)
-		(property "Description" "4 resistor network, parallel topology"
+		(property "Description" "100Ω ±5% 62.5mW 0603 Resistor Array"
 			(at 113.03 52.07 0)
 			(hide yes)
@@
 	)
 	(symbol
-		(lib_id "Device:R_Small")
+		(lib_id "Modxo-Designs:R_5k1_0603_USB")
 		(at 53.34 179.07 0)
 		(unit 1)
@@
 			)
 		)
-		(property "Description" "Resistor, small symbol"
+		(property "Description" "5.1kΩ ±1% 100mW 0603 Thick Film Resistor"
 			(at 53.34 179.07 0)
 			(hide yes)
@@
 	)
 	(symbol
-		(lib_id "Device:R_Small")
+		(lib_id "Modxo-Designs:R_27_0402_USB")
 		(at 34.29 62.23 270)
 		(unit 1)
@@
 			)
 		)
-		(property "Description" "Resistor, small symbol"
+		(property "Description" "27Ω ±1% 100mW 0603 Thick Film Resistor"
 			(at 34.29 62.23 0)
 			(hide yes)
@@
 	)
 	(symbol
-		(lib_id "Device:R_Small")
+		(lib_id "Modxo-Designs:R_27_0402_USB")
 		(at 34.29 64.77 270)
 		(mirror x)
@@
 			)
 		)
-		(property "Description" "Resistor, small symbol"
+		(property "Description" "27Ω ±1% 100mW 0603 Thick Film Resistor"
 			(at 34.29 64.77 0)
 			(hide yes)
@@
 	)
 	(symbol
-		(lib_id "Device:R_Small")
+		(lib_id "Modxo-Designs:R_5k1_0603_USB")
 		(at 45.72 179.07 0)
 		(unit 1)
@@
 			)
 		)
-		(property "Description" "Resistor, small symbol"
+		(property "Description" "5.1kΩ ±1% 100mW 0603 Thick Film Resistor"
 			(at 45.72 179.07 0)
 			(hide yes)

Commit message: Move most symbols to library
Parts:
- C1, C2: footprint Capacitor_SMD:C_0402_1005Metric -> Capacitor_SMD:C_0603_1608Metric; symbol Modxo-Designs:C_1u_0402_Decouple -> Modxo-Designs:C_1u_0603_Decouple; Distributor Link 1 https://www.digikey.com/en/products/detail/samsung-electro-mechanics/CL05A105KA5NQNC/3887103?s=N4IgTCBcDaIMIBkAMBWAggRlQaTSgcgIr5wgC6AvkA -> https://www.digikey.com/en/products/detail/samsung-electro-mechanics/CL10A105KB8NNNC/3887518; Distributor Link 2 https://www.mouser.com/ProductDetail/Samsung-Electro-Mechan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 -> https://www.mouser.com/en/ProductDetail/Samsung-Electro-Mec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; LCSC C52923 -> C1592; Manufacturer Part Number CL05A105KA5NQNC -> CL10A105KO8NNNC
- D1, D2: symbol Diode:1N5819WS -> Modxo-Designs:1N5819WS
- J1: symbol Connector_Generic:Conn_02x08_Odd_Even -> Modxo-Designs:Conn_02x08_Odd_Even_LPC
- LED1: symbol Device:LED -> Modxo-Designs:LED
- LED2: symbol LED:WS2812B-2020 -> Modxo-Designs:WS2812B-2020
- SW1: symbol Switch:SW_Push -> Modxo-Designs:SW_BOOT
- U2: symbol Memory_Flash:W25Q128JVS -> Modxo-Designs:W25Q128JVS
Changed lines of the file:
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@@
 	)
 	(symbol
-		(lib_id "Modxo-Designs:C_1u_0402_Decouple")
+		(lib_id "Modxo-Designs:C_1u_0603_Decouple")
 		(at 262.89 24.13 0)
 		(unit 1)
@@
 			)
 		)
-		(property "Footprint" "Capacitor_SMD:C_0402_1005Metric"
+		(property "Footprint" "Capacitor_SMD:C_0603_1608Metric"
 			(at 262.89 24.13 0)
 			(hide yes)
@@
 			)
 		)
-		(property "Datasheet" "https://mm.digikey.com/Volume0/opasdata/d220001/medias/docus/41/CL05A105KA5NQNC.pdf"
+		(property "Datasheet" "kicad-embed://02336ea48ea44ca18c72517dd3cb7b47.pdf"
 			(at 262.89 24.13 0)
 			(hide yes)
@@
 			)
 		)
-		(property "Description" "1uF ±10% 25V Ceramic Capacitor X5R 0402"
+		(property "Description" "1uF ±10% 16V Ceramic Capacitor X5R 0603"
 			(at 262.89 24.13 0)
 			(hide yes)
@@
 			)
 		)
-		(property "Manufacturer Part Number" "CL05A105KA5NQNC"
+		(property "Manufacturer Part Number" "CL10A105KO8NNNC"
 			(at 262.89 24.13 0)
 			(hide yes)
@@
 			)
 		)
-		(property "Distributor Link 1" "https://www.digikey.com/en/products/detail/samsung-electro-mechanics/CL05A105KA5NQNC/3887103?s=N4IgTCBcDaIMIBkAMBWAggRlQaTSgcgIr5wgC6AvkA"
+		(property "Distributor Link 1" "https://www.digikey.com/en/products/detail/samsung-electro-mechanics/CL10A105KB8NNNC/3887518"
 			(at 262.89 24.13 0)
 			(hide yes)
@@
 			)
 		)
-		(property "Distributor Link 2" "https://www.mouser.com/ProductDetail/Samsung-Electro-Mechanics/CL05A105KA5NQNC?qs=X6jEic%2FHinDIeFgZnm60Lw%3D%3D"
+		(property "Distributor Link 2" "https://www.mouser.com/en/ProductDetail/Samsung-Electro-Mechanics/CL10A105KB8NNNC?qs=ktYoCbbtCSJz4pFCLWXd5g%3D%3D"
 			(at 262.89 24.13 0)
 			(hide yes)
@@
 			)
 		)
-		(property "LCSC" "C52923"
+		(property "LCSC" "C1592"
 			(at 262.89 24.13 0)
 			(hide yes)
@@
 	)
 	(symbol
-		(lib_id "Connector_Generic:Conn_02x08_Odd_Even")
+		(lib_id "Modxo-Designs:Conn_02x08_Odd_Even_LPC")
 		(at 210.82 57.15 180)
 		(unit 1)
@@
 	)
 	(symbol
-		(lib_id "LED:WS2812B-2020")
+		(lib_id "Modxo-Designs:WS2812B-2020")
 		(at 102.87 172.72 0)
 		(unit 1)
@@
 	)
 	(symbol
-		(lib_id "Memory_Flash:W25Q128JVS")
+		(lib_id "Modxo-Designs:W25Q128JVS")
 		(at 208.28 144.78 0)
 		(unit 1)
@@
 	)
 	(symbol
-		(lib_id "Modxo-Designs:C_1u_0402_Decouple")
+		(lib_id "Modxo-Designs:C_1u_0603_Decouple")
 		(at 157.48 24.13 0)
 		(unit 1)
@@
 			)
 		)
-		(property "Footprint" "Capacitor_SMD:C_0402_1005Metric"
+		(property "Footprint" "Capacitor_SMD:C_0603_1608Metric"
 			(at 157.48 24.13 0)
 			(hide yes)
@@
 			)
 		)
-		(property "Datasheet" "https://mm.digikey.com/Volume0/opasdata/d220001/medias/docus/41/CL05A105KA5NQNC.pdf"
+		(property "Datasheet" "kicad-embed://02336ea48ea44ca18c72517dd3cb7b47.pdf"
 			(at 157.48 24.13 0)
 			(hide yes)
@@
 			)
 		)
-		(property "Description" "1uF ±10% 25V Ceramic Capacitor X5R 0402"
+		(property "Description" "1uF ±10% 16V Ceramic Capacitor X5R 0603"
 			(at 157.48 24.13 0)
 			(hide yes)
@@
 			)
 		)
-		(property "Manufacturer Part Number" "CL05A105KA5NQNC"
+		(property "Manufacturer Part Number" "CL10A105KO8NNNC"
 			(at 157.48 24.13 0)
 			(hide yes)
@@
 			)
 		)
-		(property "Distributor Link 1" "https://www.digikey.com/en/products/detail/samsung-electro-mechanics/CL05A105KA5NQNC/3887103?s=N4IgTCBcDaIMIBkAMBWAggRlQaTSgcgIr5wgC6AvkA"
+		(property "Distributor Link 1" "https://www.digikey.com/en/products/detail/samsung-electro-mechanics/CL10A105KB8NNNC/3887518"
 			(at 157.48 24.13 0)
 			(hide yes)
@@
 			)
 		)
-		(property "Distributor Link 2" "https://www.mouser.com/ProductDetail/Samsung-Electro-Mechanics/CL05A105KA5NQNC?qs=X6jEic%2FHinDIeFgZnm60Lw%3D%3D"
+		(property "Distributor Link 2" "https://www.mouser.com/en/ProductDetail/Samsung-Electro-Mechanics/CL10A105KB8NNNC?qs=ktYoCbbtCSJz4pFCLWXd5g%3D%3D"
 			(at 157.48 24.13 0)
 			(hide yes)
@@
 			)
 		)
-		(property "LCSC" "C52923"
+		(property "LCSC" "C1592"
 			(at 157.48 24.13 0)
 			(hide yes)
@@
 	)
 	(symbol
-		(lib_id "Device:LED")
+		(lib_id "Modxo-Designs:LED")
 		(at 121.92 90.17 270)
 		(mirror x)
@@
 	)
 	(symbol
-		(lib_id "Diode:1N5819WS")
+		(lib_id "Modxo-Designs:1N5819WS")
 		(at 186.69 59.69 0)
 		(unit 1)
@@
 	)
 	(symbol
-		(lib_id "Diode:1N5819WS")
+		(lib_id "Modxo-Designs:1N5819WS")
 		(at 60.96 149.86 0)
 		(mirror y)
@@
 	)
 	(symbol
-		(lib_id "Switch:SW_Push")
+		(lib_id "Modxo-Designs:SW_BOOT")
 		(at 154.94 186.69 0)
 		(unit 1)
